File: CANmodule.sch (KiCad schematic (older format))
At the start: 15 parts, among them J1 RJ45, U3 TLP2361, U4 TLP2361, U5 MCP2551-I/SN

Commit message: PCB layout
Parts:
- R201: renamed from R1; footprint Resistors_SMD:R_1210_HandSoldering -> Resistors_SMD:R_1206_HandSoldering
- R202: renamed from R2; footprint Resistors_SMD:R_1210_HandSoldering -> Resistors_SMD:R_1206_HandSoldering
- R203: renamed from R3; footprint Resistors_SMD:R_1210_HandSoldering -> Resistors_SMD:R_1206_HandSoldering
- R204: renamed from R4; footprint Resistors_SMD:R_1210_HandSoldering -> Resistors_SMD:R_1206_HandSoldering
- R205: renamed from R5; footprint Resistors_SMD:R_1210_HandSoldering -> Resistors_SMD:R_1206_HandSoldering
- gave numbers to parts that had none: 1
- renumbered C1 to C201, D1 to D201, J1 to J202, JP1 to JP201, JP2 to JP202, JP3 to JP203, U3 to U201, U4 to U202, U5 to U203
Changed lines of the file:
@@
 $EndDescr
 $Comp
-L R R3
+L R R203
 U 1 1 57FCAEE8
 P 6850 2000
-F 0 "R3" V 6930 2000 50  0000 C CNN
+F 0 "R203" V 6930 2000 50  0000 C CNN
 F 1 "4.7K" V 6850 2000 50  0000 C CNN
-F 2 "Resistors_SMD:R_1210_HandSoldering" V 6780 2000 50  0001 C CNN
+F 2 "Resistors_SMD:R_1206_HandSoldering" V 6780 2000 50  0001 C CNN
 F 3 "" H 6850 2000 50  0000 C CNN
 	1    6850 2000
@@
 $EndComp
 $Comp
-L C C1
+L C C201
 U 1 1 57FCAEE9
 P 8700 2500
-F 0 "C1" H 8725 2600 50  0000 L CNN
+F 0 "C201" H 8725 2600 50  0000 L CNN
 F 1 "4.7nF" H 8725 2400 50  0000 L CNN
 F 2 "Capacitors_SMD:C_1206" H 8738 2350 50  0001 C CNN
@@
 $EndComp
 $Comp
-L R R4
+L R R204
 U 1 1 57FCAEEA
 P 7950 2350
-F 0 "R4" V 8030 2350 50  0000 C CNN
+F 0 "R204" V 8030 2350 50  0000 C CNN
 F 1 "60" V 7950 2350 50  0000 C CNN
-F 2 "Resistors_SMD:R_1210_HandSoldering" V 7880 2350 50  0001 C CNN
+F 2 "Resistors_SMD:R_1206_HandSoldering" V 7880 2350 50  0001 C CNN
 F 3 "" H 7950 2350 50  0000 C CNN
 	1    7950 2350
@@
 $EndComp
 $Comp
-L R R5
+L R R205
 U 1 1 57FCAEEB
 P 8150 2350
-F 0 "R5" V 8230 2350 50  0000 C CNN
+F 0 "R205" V 8230 2350 50  0000 C CNN
 F 1 "60" V 8150 2350 50  0000 C CNN
-F 2 "Resistors_SMD:R_1210_HandSoldering" V 8080 2350 50  0001 C CNN
+F 2 "Resistors_SMD:R_1206_HandSoldering" V 8080 2350 50  0001 C CNN
 F 3 "" H 8150 2350 50  0000 C CNN
 	1    8150 2350
@@
 CAN_L
 $Comp
-L R R2
+L R R202
 U 1 1 57FCAEF2
 P 6300 1450
-F 0 "R2" V 6380 1450 50  0000 C CNN
+F 0 "R202" V 6380 1450 50  0000 C CNN
 F 1 "330" V 6300 1450 50  0000 C CNN
-F 2 "Resistors_SMD:R_1210_HandSoldering" V 6230 1450 50  0001 C CNN
+F 2 "Resistors_SMD:R_1206_HandSoldering" V 6230 1450 50  0001 C CNN
 F 3 "" H 6300 1450 50  0000 C CNN
 	1    6300 1450
@@
 $EndComp
 $Comp
-L Jumper_NC_Small JP1
+L Jumper_NC_Small JP201
 U 1 1 57FCAEF3
 P 7950 2000
-F 0 "JP1" H 7950 2080 50  0000 C CNN
+F 0 "JP201" H 7950 2080 50  0000 C CNN
 F 1 "Terminate" H 7960 1940 50  0001 C CNN
 F 2 "electric_car_lib:JumperSingle" H 7950 2000 50  0001 C CNN
@@
 $EndComp
 $Comp
-L Jumper_NC_Small JP2
+L Jumper_NC_Small JP202
 U 1 1 57FCAEF4
 P 8150 2000
-F 0 "JP2" H 8150 2080 50  0000 C CNN
+F 0 "JP202" H 8150 2080 50  0000 C CNN
 F 1 "Terminate" H 8160 1940 50  0000 C CNN
 F 2 "electric_car_lib:JumperSingle" H 8150 2000 50  0001 C CNN
@@
 $EndComp
 $Comp
-L Jumper_NC_Small JP3
+L Jumper_NC_Small JP203
 U 1 1 57FCAEF5
 P 8400 2500
-F 0 "JP3" H 8400 2580 50  0000 C CNN
+F 0 "JP203" H 8400 2580 50  0000 C CNN
 F 1 "Filter" H 8410 2440 50  0000 C CNN
 F 2 "electric_car_lib:JumperSingle" H 8400 2500 50  0001 C CNN
@@
 $EndComp
 $Comp
-L R R1
+L R R201
 U 1 1 57FCAEF6
 P 4800 2050
-F 0 "R1" V 4880 2050 50  0000 C CNN
+F 0 "R201" V 4880 2050 50  0000 C CNN
 F 1 "100" V 4800 2050 50  0000 C CNN
-F 2 "Resistors_SMD:R_1210_HandSoldering" V 4730 2050 50  0001 C CNN
+F 2 "Resistors_SMD:R_1206_HandSoldering" V 4730 2050 50  0001 C CNN
 F 3 "" H 4800 2050 50  0000 C CNN
 	1    4800 2050
@@
 $EndComp
 $Comp
-L TLP2361 U4
+L TLP2361 U202
 U 1 1 57FCAEF8
 P 5550 2100
-F 0 "U4" H 5550 1900 50  0000 L CNN
+F 0 "U202" H 5550 1900 50  0000 L CNN
 F 1 "TLP2361" H 5550 2300 50  0000 C CNN
 F 2 "electric_car_lib:soic-5" H 5350 1900 50  0001 L CIN
@@
 $EndComp
 $Comp
-L TLP2361 U3
+L TLP2361 U201
 U 1 1 57FCAEF9
 P 5550 1600
-F 0 "U3" H 5550 1400 50  0000 L CNN
+F 0 "U201" H 5550 1400 50  0000 L CNN
 F 1 "TLP2361" H 5550 1800 50  0000 C CNN
 F 2 "electric_car_lib:soic-5" H 5350 1400 50  0001 L CIN
@@
 CAN interface
 $Comp
-L PESD1CAN D1
+L PESD1CAN D201
 U 1 1 57FCAEFA
 P 8700 1500
-F 0 "D1" H 8700 1250 60  0000 C CNN
+F 0 "D201" H 8700 1250 60  0000 C CNN
 F 1 "PESD1CAN" H 8650 1800 60  0000 C CNN
 F 2 "TO_SOT_Packages_SMD:SOT-23_Handsoldering" H 8700 1500 60  0001 C CNN
@@
 $EndComp
 $Comp
-L MCP2551-I/SN U5
+L MCP2551-I/SN U203
 U 1 1 57FCAEFB
 P 7200 1500
-F 0 "U5" H 6800 1850 50  0000 L CNN
+F 0 "U203" H 6800 1850 50  0000 L CNN
 F 1 "MCP2551-I/SN" H 7300 1850 50  0000 L CNN
 F 2 "Power_Integrations:SO-8" H 7200 1500 50  0000 C CIN
@@
 CAN_RX
 $Comp
-L RJ45 J1
+L RJ45 J202
 U 1 1 57FCC775
 P 8000 4050
-F 0 "J1" H 8020 4070 20  0000 C CNN
+F 0 "J202" H 8020 4070 20  0000 C CNN
 F 1 "RJ45" H 7850 4550 50  0000 C CNN
 F 2 "Connect:RJ45_8" H 8000 4050 50  0001 C CNN
@@
 	8250 4800 8250 4500
 $Comp
-L RJ45 J?
+L RJ45 J201
 U 1 1 5821749D
 P 6700 4050
-F 0 "J?" H 6720 4070 20  0000 C CNN
+F 0 "J201" H 6720 4070 20  0000 C CNN
 F 1 "RJ45" H 6550 4550 50  0000 C CNN
 F 2 "Connect:RJ45_8" H 6700 4050 50  0001 C CNN
